Commit message: add serial

File: ros2_control_demo_description/diffbot_description/ros2_control/diffbot_system.ros2_control.xacro (robot description, xacro)
@@ -13,4 +13,5 @@
           <param name="example_param_hw_start_duration_sec">2.0</param>
           <param name="example_param_hw_stop_duration_sec">3.0</param>
+          <param name="example_param_hw_slowdown">2.0</param>
         </xacro:unless>
       </hardware>

File: ros2_control_demo_description/diffbot_description/urdf/diffbot.urdf.xacro (robot description, xacro)
@@ -1,161 +1,190 @@
 <?xml version="1.0"?>
-<robot xmlns:xacro="http://www.ros.org/wiki/xacro">
+<robot name="diffdrive_robot" xmlns:xacro="http://ros.org/wiki/xacro">
   <xacro:macro name="diffbot" params="prefix">
-  <!-- Constants for robot dimensions -->
-  <xacro:property name="PI" value="3.1415926535897931"/>
-  <xacro:property name="base_mass" value="0.3" /> <!-- arbitrary value for base mass -->
-  <xacro:property name="base_width" value="0.1" />
-  <xacro:property name="base_length" value="0.1" />
-  <xacro:property name="base_height" value="0.05" />
-  <xacro:property name="wheel_mass" value="0.3" /> <!-- arbitrary value for wheel mass -->
-  <xacro:property name="wheel_len" value="0.020" />
-  <xacro:property name="wheel_radius" value="0.015" />
-  <xacro:property name="caster_wheel_mass" value="0.1" /> <!-- arbitrary value for caster wheel mass -->
-  <xacro:property name="caster_wheel_radius" value="0.015" />
-  <xacro:property name="z_offset" value="-${base_height/2}" /> <!-- Space btw top of beam and the each joint -->
-  <!-- Base Link -->
-  <link name="${prefix}base_link">
-    <collision>
-      <origin xyz="0 0 0" rpy="0 0 0"/>
-      <geometry>
-        <box size="${base_width} ${base_length} ${base_height}"/>
-      </geometry>
-    </collision>
-    <visual>
-      <origin xyz="0 0 0" rpy="0 0 0"/>
-      <geometry>
-        <box size="${base_width} ${base_length} ${base_height}"/>
-      </geometry>
-      <material name="orange"/>
-    </visual>
-    <inertial>
-      <origin xyz="0 0 0" rpy="0 0 0"/>
-      <mass value="${base_mass}"/>
-      <inertia
-        ixx="${base_mass / 12.0 * (base_length*base_length + base_height*base_height)}" ixy="0.0" ixz="0.0"
-        iyy="${base_mass / 12.0 * (base_height*base_height + base_width*base_width)}" iyz="0.0"
-        izz="${base_mass / 12.0 * (base_width*base_width + base_length*base_length)}"/>
+    <!-- Constants for robot dimensions -->
+    <xacro:property name="PI" value="3.1415926535897931" />
+    <xacro:property name="base_mass" value="0.3" /> <!-- arbitrary value for base mass -->
+    <xacro:property name="base_width" value="0.1" />
+    <xacro:property name="base_length" value="0.1" />
+    <xacro:property name="base_height" value="0.05" />
+    <xacro:property name="wheel_mass" value="0.3" /> <!-- arbitrary value for wheel mass -->
+    <xacro:property name="wheel_len" value="0.020" />
+    <xacro:property name="wheel_radius" value="0.015" />
+    <xacro:property name="caster_wheel_mass" value="0.1" /> <!-- arbitrary value for caster wheel mass -->
+    <xacro:property name="caster_wheel_radius" value="0.015" />
+    <xacro:property name="z_offset" value="-${base_height/2}" /> <!-- Space btw top of beam and the each joint -->
+    <xacro:property name="wheel_zoff" value="0.01"/>
+    <!-- Define some commonly used intertial properties  -->
+    <xacro:macro name="box_inertia" params="m w h d">
+      <inertial>
+        <origin xyz="0 0 0" rpy="${pi/2} 0 ${pi/2}"/>
+        <mass value="${m}"/>
+        <inertia ixx="${(m/12) * (h*h + d*d)}" ixy="0.0" ixz="0.0" iyy="${(m/12) * (w*w + d*d)}" iyz="0.0" izz="${(m/12) * (w*w + h*h)}"/>
+      </inertial>
+    </xacro:macro>
+    <!-- Base Link -->
+    <link name="${prefix}base_link">
+      <collision>
+        <origin xyz="0 0 0" rpy="0 0 0" />
+        <geometry>
+          <box size="${base_width} ${base_length} ${base_height}" />
+        </geometry>
+      </collision>
+      <visual>
+        <origin xyz="0 0 0" rpy="0 0 0" />
+        <geometry>
+          <box size="${base_width} ${base_length} ${base_height}" />
+        </geometry>
+        <material name="orange" />
+      </visual>
+      <inertial>
+        <origin xyz="0 0 0" rpy="0 0 0" />
+        <mass value="${base_mass}" />
+        <inertia ixx="${base_mass / 12.0 * (base_length*base_length + base_height*base_height)}" ixy="0.0" ixz="0.0" iyy="${base_mass / 12.0 * (base_height*base_height + base_width*base_width)}" iyz="0.0" izz="${base_mass / 12.0 * (base_width*base_width + base_length*base_length)}" />
       </inertial>
     </link>
+    <!-- Robot Footprint -->
+    <link name="${prefix}base_footprint">
+  	  <xacro:box_inertia m="0" w="0" d="0" h="0"/>
+    </link>
+    <joint name="${prefix}base_joint" type="fixed">
+      <parent link="${prefix}base_link"/>
+      <child link="${prefix}base_footprint"/>
+      <origin xyz="0.0 0.0 ${-(wheel_radius+wheel_zoff)}" rpy="0 0 0"/>
+    </joint>
     <joint name="${prefix}left_wheel_joint" type="continuous">
-      <parent link="${prefix}base_link"/>
-      <child link="${prefix}left_wheel"/>
-      <origin xyz="0 -${base_width/2} ${z_offset}" rpy="0 0 0"/>
-      <axis xyz="0 1 0"/>
-      <dynamics damping="0.2"/>
+      <parent link="${prefix}base_link" />
+      <child link="${prefix}left_wheel" />
+      <origin xyz="0 -${base_width/2} ${z_offset}" rpy="0 0 0" />
+      <axis xyz="0 1 0" />
+      <dynamics damping="0.2" />
     </joint>
     <!-- left wheel Link -->
     <link name="${prefix}left_wheel">
       <collision>
-        <origin xyz="0 0 0" rpy="${PI/2} 0 0"/>
+        <origin xyz="0 0 0" rpy="${PI/2} 0 0" />
         <geometry>
-          <cylinder length="${wheel_len}" radius="${wheel_radius}"/>
+          <cylinder length="${wheel_len}" radius="${wheel_radius}" />
         </geometry>
       </collision>
       <visual>
-        <origin xyz="0 0 0" rpy="${PI/2} 0 0"/>
+        <origin xyz="0 0 0" rpy="${PI/2} 0 0" />
         <geometry>
-          <cylinder length="${wheel_len}" radius="${wheel_radius}"/>
+          <cylinder length="${wheel_len}" radius="${wheel_radius}" />
         </geometry>
-        <material name="black"/>
+        <material name="black" />
       </visual>
       <inertial>
-        <origin xyz="0 0 0" rpy="${PI/2} 0 0"/>
-        <mass value="${wheel_mass}"/>
-        <inertia
-          ixx="${wheel_mass / 12.0 * (3*wheel_radius + wheel_len*wheel_len)}" ixy="0.0" ixz="0.0"
-          iyy="${wheel_mass / 12.0 * wheel_radius*wheel_radius}" iyz="0.0"
-          izz="${wheel_mass / 12.0 * wheel_radius*wheel_radius}"/>
-        </inertial>
-      </link>
+        <origin xyz="0 0 0" rpy="${PI/2} 0 0" />
+        <mass value="${wheel_mass}" />
+        <inertia ixx="${wheel_mass / 12.0 * (3*wheel_radius + wheel_len*wheel_len)}" ixy="0.0" ixz="0.0" iyy="${wheel_mass / 12.0 * wheel_radius*wheel_radius}" iyz="0.0" izz="${wheel_mass / 12.0 * wheel_radius*wheel_radius}" />
+      </inertial>
+    </link>
     <joint name="${prefix}right_wheel_joint" type="continuous">
-      <parent link="${prefix}base_link"/>
-      <child link="${prefix}right_wheel"/>
-      <origin xyz="0 ${base_width/2} ${z_offset}" rpy="0 0 0"/>
-      <axis xyz="0 1 0"/>
-      <dynamics damping="0.2"/>
+      <parent link="${prefix}base_link" />
+      <child link="${prefix}right_wheel" />
+      <origin xyz="0 ${base_width/2} ${z_offset}" rpy="0 0 0" />
+      <axis xyz="0 1 0" />
+      <dynamics damping="0.2" />
     </joint>
     <!-- right wheel Link -->
     <link name="${prefix}right_wheel">
       <collision>
-        <origin xyz="0 0 0" rpy="${PI/2} 0 0"/>
+        <origin xyz="0 0 0" rpy="${PI/2} 0 0" />
         <geometry>
-          <cylinder length="${wheel_len}" radius="${wheel_radius}"/>
+          <cylinder length="${wheel_len}" radius="${wheel_radius}" />
         </geometry>
       </collision>
       <visual>
-        <origin xyz="0 0 0" rpy="${PI/2} 0 0"/>
+        <origin xyz="0 0 0" rpy="${PI/2} 0 0" />
         <geometry>
-          <cylinder length="${wheel_len}" radius="${wheel_radius}"/>
+          <cylinder length="${wheel_len}" radius="${wheel_radius}" />
         </geometry>
-        <material name="black"/>
+        <material name="black" />
       </visual>
       <inertial>
-        <origin xyz="0 0 0" rpy="${PI/2} 0 0"/>
-        <mass value="${wheel_mass}"/>
-        <inertia
-          ixx="${wheel_mass / 12.0 * (3*wheel_radius + wheel_len*wheel_len)}" ixy="0.0" ixz="0.0"
-          iyy="${wheel_mass / 12.0 * wheel_radius*wheel_radius}" iyz="0.0"
-          izz="${wheel_mass / 12.0 * wheel_radius*wheel_radius}"/>
-        </inertial>
-      </link>
+        <origin xyz="0 0 0" rpy="${PI/2} 0 0" />
+        <mass value="${wheel_mass}" />
+        <inertia ixx="${wheel_mass / 12.0 * (3*wheel_radius + wheel_len*wheel_len)}" ixy="0.0" ixz="0.0" iyy="${wheel_mass / 12.0 * wheel_radius*wheel_radius}" iyz="0.0" izz="${wheel_mass / 12.0 * wheel_radius*wheel_radius}" />
+      </inertial>
+    </link>
     <joint name="${prefix}caster_frontal_wheel_joint" type="fixed">
-      <parent link="${prefix}base_link"/>
-      <child link="${prefix}caster_frontal_wheel"/>
-      <origin xyz="${base_width/2 - caster_wheel_radius} 0 ${z_offset}" rpy="0 0 0"/>
+      <parent link="${prefix}base_link" />
+      <child link="${prefix}caster_frontal_wheel" />
+      <origin xyz="${base_width/2 - caster_wheel_radius} 0 ${z_offset}" rpy="0 0 0" />
     </joint>
     <!-- caster frontal wheel Link -->
     <link name="${prefix}caster_frontal_wheel">
       <collision>
-        <origin xyz="0 0 0" rpy="0 0 0"/>
+        <origin xyz="0 0 0" rpy="0 0 0" />
         <geometry>
-          <sphere radius="${caster_wheel_radius}"/>
+          <sphere radius="${caster_wheel_radius}" />
         </geometry>
       </collision>
       <visual>
-        <origin xyz="0 0 0" rpy="0 0 0"/>
+        <origin xyz="0 0 0" rpy="0 0 0" />
         <geometry>
-          <sphere radius="${caster_wheel_radius}"/>
+          <sphere radius="${caster_wheel_radius}" />
         </geometry>
-        <material name="white"/>
+        <material name="white" />
       </visual>
       <inertial>
-        <origin xyz="0 0 0" rpy="0 0 0"/>
-        <mass value="${caster_wheel_mass}"/>
-        <inertia
-          ixx="${caster_wheel_mass * 0.4 * (caster_wheel_radius * caster_wheel_radius)}" ixy="0.0" ixz="0.0"
-          iyy="${caster_wheel_mass * 0.4 * (caster_wheel_radius * caster_wheel_radius)}" iyz="0.0"
-          izz="${caster_wheel_mass * 0.4 * (caster_wheel_radius * caster_wheel_radius)}"/>
-        </inertial>
-      </link>
+        <origin xyz="0 0 0" rpy="0 0 0" />
+        <mass value="${caster_wheel_mass}" />
+        <inertia ixx="${caster_wheel_mass * 0.4 * (caster_wheel_radius * caster_wheel_radius)}" ixy="0.0" ixz="0.0" iyy="${caster_wheel_mass * 0.4 * (caster_wheel_radius * caster_wheel_radius)}" iyz="0.0" izz="${caster_wheel_mass * 0.4 * (caster_wheel_radius * caster_wheel_radius)}" />
+      </inertial>
+    </link>
     <joint name="${prefix}caster_rear_wheel_joint" type="fixed">
-      <parent link="${prefix}base_link"/>
-      <child link="${prefix}caster_rear_wheel"/>
-      <origin xyz="${-base_width/2 + caster_wheel_radius} 0 ${z_offset}" rpy="0 0 0"/>
+      <parent link="${prefix}base_link" />
+      <child link="${prefix}caster_rear_wheel" />
+      <origin xyz="${-base_width/2 + caster_wheel_radius} 0 ${z_offset}" rpy="0 0 0" />
     </joint>
     <!-- caster rear wheel Link -->
     <link name="${prefix}caster_rear_wheel">
       <collision>
-        <origin xyz="0 0 0" rpy="0 0 0"/>
+        <origin xyz="0 0 0" rpy="0 0 0" />
         <geometry>
-          <sphere radius="${caster_wheel_radius}"/>
+          <sphere radius="${caster_wheel_radius}" />
         </geometry>
       </collision>
       <visual>
-        <origin xyz="0 0 0" rpy="0 0 0"/>
+        <origin xyz="0 0 0" rpy="0 0 0" />
         <geometry>
-          <sphere radius="${caster_wheel_radius}"/>
+          <sphere radius="${caster_wheel_radius}" />
         </geometry>
-        <material name="white"/>
+        <material name="white" />
       </visual>
       <inertial>
-        <origin xyz="0 0 0" rpy="0 0 0"/>
-        <mass value="${caster_wheel_mass}"/>
-        <inertia
-          ixx="${caster_wheel_mass * 0.4 * (caster_wheel_radius * caster_wheel_radius)}" ixy="0.0" ixz="0.0"
-          iyy="${caster_wheel_mass * 0.4 * (caster_wheel_radius * caster_wheel_radius)}" iyz="0.0"
-          izz="${caster_wheel_mass * 0.4 * (caster_wheel_radius * caster_wheel_radius)}"/>
-        </inertial>
-      </link>
+        <origin xyz="0 0 0" rpy="0 0 0" />
+        <mass value="${caster_wheel_mass}" />
+        <inertia ixx="${caster_wheel_mass * 0.4 * (caster_wheel_radius * caster_wheel_radius)}" ixy="0.0" ixz="0.0" iyy="${caster_wheel_mass * 0.4 * (caster_wheel_radius * caster_wheel_radius)}" iyz="0.0" izz="${caster_wheel_mass * 0.4 * (caster_wheel_radius * caster_wheel_radius)}" />
+      </inertial>
+    </link>
   </xacro:macro>
+  <!--
+<ros2_control name="diffbot_system" type="system">
+  <hardware>
+    <plugin>ros2_control_demo_hardware/DiffBotSystemHardware</plugin>
+    <param name="example_param_hw_start_duration_sec">2.0</param>
+    <param name="example_param_hw_stop_duration_sec">3.0</param>
+    <param name="example_param_hw_slowdown">2.0</param>
+  </hardware>
+  <joint name="left_wheel_joint">
+    <command_interface name="velocity">
+      <param name="min">-1</param>
+      <param name="max">1</param>
+    </command_interface>
+    <state_interface name="position"/>
+    <state_interface name="velocity"/>
+  </joint>
+  <joint name="right_wheel_joint">
+    <command_interface name="velocity">
+      <param name="min">-1</param>
+      <param name="max">1</param>
+    </command_interface>
+    <state_interface name="position"/>
+    <state_interface name="velocity"/>
+  </joint>
+</ros2_control>
+-->
 </robot>

File: ros2_control_demo_description/diffbot_description/urdf/diffbot_system.urdf.xacro (robot description, xacro)
@@ -5,8 +5,8 @@
 https://github.com/ros-simulation/gazebo_ros_demos/blob/kinetic-devel/diffbot_description/urdf/diffbot.xacro
 -->
-<robot xmlns:xacro="http://www.ros.org/wiki/xacro" name="diffdrive_robot">
+<robot name="diffdrive_robot" xmlns:xacro="http://ros.org/wiki/xacro">
   <xacro:arg name="use_sim" default="false" />
   <!-- Enable setting arguments from the launch file -->
-  <xacro:arg name="use_fake_hardware" default="true" />
+  <xacro:arg name="use_fake_hardware" default="false" />
   <xacro:arg name="fake_sensor_commands" default="false" />
   <xacro:arg name="prefix" default="" />
@@ -20,7 +20,11 @@
   <xacro:diffbot prefix="$(arg prefix)" />
   <xacro:diffbot_gazebo prefix="$(arg prefix)" />
-  <xacro:diffbot_system
-    name="DiffBotSystem" prefix="$(arg prefix)"
-    use_fake_hardware="$(arg use_fake_hardware)"
-    fake_sensor_commands="$(arg fake_sensor_commands)"/>
+  <xacro:diffbot_system name="DiffBotSystem" prefix="$(arg prefix)" use_fake_hardware="$(arg use_fake_hardware)" fake_sensor_commands="$(arg fake_sensor_commands)" />
+  <!--
+<ros2_control name="rotate_box_bot" type="system">
+  <hardware>
+    <plugin>test_system</plugin>
+  </hardware>
+</ros2_control>
+-->
 </robot>
